File: examples/butterworth/butterworth.sch (KiCad schematic (older format))
At the start: 10 parts, among them U101 LMV981

Commit message: Update the butterworth example
Add and use LMH6624 OP-amp in butterworth schema

Xyce gives a "timestamp too small" error with LMV681.
Use LMH6624 instead and clean up the schematic a bit.

Start using a prerendered HTML page as an example of the notebook
use instead of keeping the data in the notebook.

Move the notebook and results into the examples/butterworth directory.
Parts:
- removed U101: LMV981, Package_TO_SOT_SMD:SOT-363_SC-70-6, symbol Amplifier_Operational:LMV601
- added U101: LMH6624, Package_TO_SOT_SMD:TSOT-23-5, symbol Amplifier_Operational:AD8603
Connections:
- wire segments 33 -> 30
Changed lines of the file:
@@
 Wire Wire Line
 	4600 3700 4500 3700
-Text GLabel 7350 3800 2    50   Output ~ 0
+Text GLabel 7300 3800 2    50   Output ~ 0
 VOUT
 Wire Wire Line
-	7350 3800 7100 3800
+	7300 3800 7100 3800
 $Comp
 L Device:C C102
@@
 $EndComp
 $Comp
-L Amplifier_Operational:LMV601 U101
-U 1 1 5B71E57A
-P 5900 3800
-F 0 "U101" H 6100 4150 50  0000 L CNN
-F 1 "LMV981" H 6100 4050 50  0000 L CNN
-F 2 "Package_TO_SOT_SMD:SOT-363_SC-70-6" H 5900 3800 50  0001 L CNN
-F 3 "http://www.ti.com/lit/ds/symlink/lmv601.pdf" H 5900 3450 50  0001 L CNN
-F 4 "X" H 5900 3800 50  0001 C CNN "Spice_Primitive"
-F 5 "LMV981" H 5900 3800 50  0001 C CNN "Spice_Model"
-F 6 "Y" H 5900 3800 50  0001 C CNN "Spice_Netlist_Enabled"
-F 7 "1 3 6 2 4 5" H 5900 3800 50  0001 C CNN "Spice_Node_Sequence"
-F 8 "LMV981.MOD" H 5900 3800 50  0001 C CNN "Spice_Lib_File"
-	1    5900 3800
-	1    0    0    -1
-$EndComp
-Wire Wire Line
-	5900 4100 6000 4100
-Wire Wire Line
-	6000 3500 5800 3500
-Wire Wire Line
-	6000 3500 6000 4100
-Connection ~ 5800 3500
-$Comp
 L pspice:VSOURCE V101
 U 1 1 5B747B28
@@
 Text Label 3800 3700 0    50   ~ 0
 VIN
+$Comp
+L Amplifier_Operational:AD8603 U101
+U 1 1 5B861DA4
+P 5900 3800
+F 0 "U101" H 6000 4100 50  0000 L CNN
+F 1 "LMH6624" H 6000 4000 50  0000 L CNN
+F 2 "Package_TO_SOT_SMD:TSOT-23-5" H 5900 3800 50  0001 C CNN
+F 3 "http://www.analog.com/media/en/technical-documentation/data-sheets/AD8603_8607_8609.pdf" H 5900 4000 50  0001 C CNN
+F 4 "X" H 5900 3800 50  0001 C CNN "Spice_Primitive"
+F 5 "LMH6624" H 5900 3800 50  0001 C CNN "Spice_Model"
+F 6 "Y" H 5900 3800 50  0001 C CNN "Spice_Netlist_Enabled"
+F 7 "3 4 5 2 1" H 5900 3800 50  0001 C CNN "Spice_Node_Sequence"
+F 8 "LMH6624.MOD" H 5900 3800 50  0001 C CNN "Spice_Lib_File"
+	1    5900 3800
+	1    0    0    -1
+$EndComp
 $EndSCHEMATC
